File: kicad/zxRebornClock/zxRebornClock.kicad_sch (KiCad schematic)
At the start: 101 parts, among them J1 Conn_01x04, J2 Conn_01x03, J3 USB_B_Micro, J4 Conn_01x03, J5 Jack DC, J6 Conn_01x02, Q1 MMBTA42, Q11 MMBTA42, Q2 MMBTA42, Q3 MMBTA42, Q4 MMBTA42, Q5 MMBTA42, Q6 MMBTA42, Q7 MMBTA42, Q8 MMBTA42, Q9 MMBTA42, SW1 HH, SW2 MM, SW3 SS, SW4 F, SW5 D, SW6 RESET, U1 TLP627, U2 TLP627, U3 TLP627, U4 TLP627, U6 DS1302, U7 ESP-12F, U8 USBLC6-4SC6, U9 AMS1117-3.3, Y1 32768

Commit message: renaming
Parts:
- renumbered C6 to C1, C3 to C2, C2 to C3, C1 to C6, D5 to D1, D1 to D2, D2 to D3, D3 to D4, D4 to D5, J5 to J1, J3 to J2, J1 to J3, J2 to J4, J4 to J5, Q11 to Q1, Q9 to Q10, Q1 to Q2, Q2 to Q3, Q3 to Q4, Q4 to Q5, Q5 to Q6, Q6 to Q7, Q7 to Q8, Q8 to Q9, R49 to R1, R7 to R10, R9 to R11, R44 to R12, R45 to R13, R46 to R14, R47 to R15, R10 to R16, R24 to R17, R26 to R18, R28 to R19, R1 to R2, R30 to R20, R23 to R21, R25 to R22, R27 to R23, R29 to R24, R31 to R25, R36 to R26, R37 to R27, R12 to R28, R48 to R29, R2 to R3, R40 to R30, R41 to R31, R42 to R32, R43 to R33, R38 to R34, R22 to R35, R21 to R36, R20 to R37, R19 to R38, R18 to R39, R17 to R40, R16 to R41, R15 to R42, R14 to R43, R13 to R44, R32 to R45, R33 to R46, R34 to R47, R35 to R48, R50 to R49, R6 to R5, R39 to R50, R8 to R6, R11 to R7, R3 to R8, R5 to R9, SW6 to SW1, SW5 to SW2, SW1 to SW3, SW2 to SW4, SW3 to SW5, SW4 to SW6, U5 to U1, U4 to U10, U9 to U2, U10 to U3, U8 to U4, U6 to U5, U7 to U6, U1 to U7, U2 to U8, U3 to U9, VL3 to VL2, VL2 to VL3

Commit message: add some ground symbol fixes
Other:
- moved on the sheet: J2, U3

Commit message: begin footprint setting
Parts:
- D2, D3, D4, D5: footprint (none) -> LED_SMD:LED_0805_2012Metric_Pad1.15x1.40mm_HandSolder
- R10, R11, R12, R13, R14, R15, R16, R17, R18, R19, R2, R20, R21, R22, R23, R24, R25, R26, R27, R28, R29, R3, R30, R31, R32, R33, R34, R35, R36, R37, R38, R39, R4, R40, R41, R42, R43, R44, R45, R46, R47, R48, R49, R5, R50, R6, R7, R8, R9: footprint (none) -> Resistor_SMD:R_0805_2012Metric_Pad1.20x1.40mm_HandSolder
Changed lines of the file:
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@@
 			)
 		)
-		(property "Footprint" ""
+		(property "Footprint" "Resistor_SMD:R_0805_2012Metric_Pad1.20x1.40mm_HandSolder"
 			(at 120.65 105.918 90)
 			(effects
@@
 			)
 		)
-		(property "Footprint" ""
+		(property "Footprint" "Resistor_SMD:R_0805_2012Metric_Pad1.20x1.40mm_HandSolder"
 			(at 90.17 86.868 90)
 			(effects
@@
 			)
 		)
-		(property "Footprint" ""
+		(property "Footprint" "Resistor_SMD:R_0805_2012Metric_Pad1.20x1.40mm_HandSolder"
 			(at 187.96 75.692 90)
 			(effects
@@
 			)
 		)
-		(property "Footprint" ""
+		(property "Footprint" "Resistor_SMD:R_0805_2012Metric_Pad1.20x1.40mm_HandSolder"
 			(at 134.62 212.852 90)
 			(effects
@@
 			)
 		)
-		(property "Footprint" ""
+		(property "Footprint" "Resistor_SMD:R_0805_2012Metric_Pad1.20x1.40mm_HandSolder"
 			(at 172.72 230.632 90)
 			(effects
@@
 			)
 		)
-		(property "Footprint" ""
+		(property "Footprint" "Resistor_SMD:R_0805_2012Metric_Pad1.20x1.40mm_HandSolder"
 			(at 187.96 124.968 90)
 			(effects
@@
 			)
 		)
-		(property "Footprint" ""
+		(property "Footprint" "Resistor_SMD:R_0805_2012Metric_Pad1.20x1.40mm_HandSolder"
 			(at 120.65 124.968 90)
 			(effects
@@
 			)
 		)
-		(property "Footprint" ""
+		(property "Footprint" "Resistor_SMD:R_0805_2012Metric_Pad1.20x1.40mm_HandSolder"
 			(at 187.96 96.012 90)
 			(effects
@@
 			)
 		)
-		(property "Footprint" ""
+		(property "Footprint" "Resistor_SMD:R_0805_2012Metric_Pad1.20x1.40mm_HandSolder"
 			(at 126.238 127 90)
 			(effects
@@
 			)
 		)
-		(property "Footprint" ""
+		(property "Footprint" "Resistor_SMD:R_0805_2012Metric_Pad1.20x1.40mm_HandSolder"
 			(at 187.96 119.888 90)
 			(effects
@@
 			)
 		)
-		(property "Footprint" ""
+		(property "Footprint" "Resistor_SMD:R_0805_2012Metric_Pad1.20x1.40mm_HandSolder"
 			(at 126.238 107.95 90)
 			(effects
@@
 			)
 		)
-		(property "Footprint" ""
+		(property "Footprint" "Resistor_SMD:R_0805_2012Metric_Pad1.20x1.40mm_HandSolder"
 			(at 187.96 90.932 90)
 			(effects
@@
 			)
 		)
-		(property "Footprint" ""
+		(property "Footprint" "Resistor_SMD:R_0805_2012Metric_Pad1.20x1.40mm_HandSolder"
 			(at 188.595 207.772 90)
 			(effects
@@
 			)
 		)
-		(property "Footprint" ""
+		(property "Footprint" "Resistor_SMD:R_0805_2012Metric_Pad1.20x1.40mm_HandSolder"
 			(at 95.758 127 90)
 			(effects
@@
 			)
 		)
-		(property "Footprint" ""
+		(property "Footprint" "Resistor_SMD:R_0805_2012Metric_Pad1.20x1.40mm_HandSolder"
 			(at 126.238 69.85 90)
 			(effects
@@
 			)
 		)
-		(property "Footprint" ""
+		(property "Footprint" "Resistor_SMD:R_0805_2012Metric_Pad1.20x1.40mm_HandSolder"
 			(at 154.94 189.738 90)
 			(effects
@@
 			)
 		)
-		(property "Footprint" ""
+		(property "Footprint" "Resistor_SMD:R_0805_2012Metric_Pad1.20x1.40mm_HandSolder"
 			(at 154.94 196.088 90)
 			(effects
@@
 			)
 		)
-		(property "Footprint" ""
+		(property "Footprint" "LED_SMD:LED_0805_2012Metric_Pad1.15x1.40mm_HandSolder"
 			(at 122.555 194.945 0)
 			(effects
@@
 			)
 		)
-		(property "Footprint" ""
+		(property "Footprint" "Resistor_SMD:R_0805_2012Metric_Pad1.20x1.40mm_HandSolder"
 			(at 95.758 69.85 90)
 			(effects
@@
 			)
 		)
-		(property "Footprint" ""
+		(property "Footprint" "Resistor_SMD:R_0805_2012Metric_Pad1.20x1.40mm_HandSolder"
 			(at 90.17 124.968 90)
 			(effects
@@
 			)
 		)
-		(property "Footprint" ""
+		(property "Footprint" "Resistor_SMD:R_0805_2012Metric_Pad1.20x1.40mm_HandSolder"
 			(at 187.96 80.772 90)
 			(effects
@@
 			)
 		)
-		(property "Footprint" ""
+		(property "Footprint" "Resistor_SMD:R_0805_2012Metric_Pad1.20x1.40mm_HandSolder"
 			(at 187.96 106.172 90)
 			(effects
@@
 			)
 		)
-		(property "Footprint" ""
+		(property "Footprint" "Resistor_SMD:R_0805_2012Metric_Pad1.20x1.40mm_HandSolder"
 			(at 154.94 170.688 90)
 			(effects
@@
 			)
 		)
-		(property "Footprint" ""
+		(property "Footprint" "Resistor_SMD:R_0805_2012Metric_Pad1.20x1.40mm_HandSolder"
 			(at 95.758 107.95 90)
 			(effects
@@
 			)
 		)
-		(property "Footprint" ""
+		(property "Footprint" "Resistor_SMD:R_0805_2012Metric_Pad1.20x1.40mm_HandSolder"
 			(at 154.94 177.038 90)
 			(effects
@@
 			)
 		)
-		(property "Footprint" ""
+		(property "Footprint" "Resistor_SMD:R_0805_2012Metric_Pad1.20x1.40mm_HandSolder"
 			(at 187.96 85.852 90)
 			(effects
@@
 			)
 		)
-		(property "Footprint" ""
+		(property "Footprint" "LED_SMD:LED_0805_2012Metric_Pad1.15x1.40mm_HandSolder"
 			(at 122.555 176.53 0)
 			(effects
@@
 			)
 		)
-		(property "Footprint" ""
+		(property "Footprint" "Resistor_SMD:R_0805_2012Metric_Pad1.20x1.40mm_HandSolder"
 			(at 187.96 130.048 90)
 			(effects
@@
 			)
 		)
-		(property "Footprint" ""
+		(property "Footprint" "Resistor_SMD:R_0805_2012Metric_Pad1.20x1.40mm_HandSolder"
 			(at 126.238 88.9 90)
 			(effects
@@
 			)
 		)
-		(property "Footprint" ""
+		(property "Footprint" "LED_SMD:LED_0805_2012Metric_Pad1.15x1.40mm_HandSolder"
 			(at 122.555 182.88 0)
 			(effects
@@
 			)
 		)
-		(property "Footprint" ""
+		(property "Footprint" "Resistor_SMD:R_0805_2012Metric_Pad1.20x1.40mm_HandSolder"
 			(at 126.238 146.05 90)
 			(effects
@@
 			)
 		)
-		(property "Footprint" ""
+		(property "Footprint" "Resistor_SMD:R_0805_2012Metric_Pad1.20x1.40mm_HandSolder"
 			(at 90.17 67.818 90)
 			(effects
@@
 			)
 		)
-		(property "Footprint" ""
+		(property "Footprint" "Resistor_SMD:R_0805_2012Metric_Pad1.20x1.40mm_HandSolder"
 			(at 134.62 207.772 90)
 			(effects
@@
 			)
 		)
-		(property "Footprint" ""
+		(property "Footprint" "Resistor_SMD:R_0805_2012Metric_Pad1.20x1.40mm_HandSolder"
 			(at 187.96 135.128 90)
 			(effects
@@
 			)
 		)
-		(property "Footprint" ""
+		(property "Footprint" "Resistor_SMD:R_0805_2012Metric_Pad1.20x1.40mm_HandSolder"
 			(at 187.96 101.092 90)
 			(effects
@@
 			)
 		)
-		(property "Footprint" ""
+		(property "Footprint" "Resistor_SMD:R_0805_2012Metric_Pad1.20x1.40mm_HandSolder"
 			(at 187.96 65.532 90)
 			(effects
@@
 			)
 		)
-		(property "Footprint" ""
+		(property "Footprint" "Resistor_SMD:R_0805_2012Metric_Pad1.20x1.40mm_HandSolder"
 			(at 114.935 184.658 90)
 			(effects
@@
 			)
 		)
-		(property "Footprint" ""
+		(property "Footprint" "Resistor_SMD:R_0805_2012Metric_Pad1.20x1.40mm_HandSolder"
 			(at 95.758 146.05 90)
 			(effects
@@
 			)
 		)
-		(property "Footprint" ""
+		(property "Footprint" "LED_SMD:LED_0805_2012Metric_Pad1.15x1.40mm_HandSolder"
 			(at 122.555 189.23 0)
 			(effects
@@
 			)
 		)
-		(property "Footprint" ""
+		(property "Footprint" "Resistor_SMD:R_0805_2012Metric_Pad1.20x1.40mm_HandSolder"
 			(at 154.94 183.388 90)
 			(effects
@@
 			)
 		)
-		(property "Footprint" ""
+		(property "Footprint" "Resistor_SMD:R_0805_2012Metric_Pad1.20x1.40mm_HandSolder"
 			(at 188.595 212.852 90)
 			(effects
@@
 			)
 		)
-		(property "Footprint" ""
+		(property "Footprint" "Resistor_SMD:R_0805_2012Metric_Pad1.20x1.40mm_HandSolder"
 			(at 120.65 86.868 90)
 			(effects
@@
 			)
 		)
-		(property "Footprint" ""
+		(property "Footprint" "Resistor_SMD:R_0805_2012Metric_Pad1.20x1.40mm_HandSolder"
 			(at 120.65 67.818 90)
 			(effects
@@
 			)
 		)
-		(property "Footprint" ""
+		(property "Footprint" "Resistor_SMD:R_0805_2012Metric_Pad1.20x1.40mm_HandSolder"
 			(at 114.935 191.008 90)
 			(effects
@@
 			)
 		)
-		(property "Footprint" ""
+		(property "Footprint" "Resistor_SMD:R_0805_2012Metric_Pad1.20x1.40mm_HandSolder"
 			(at 95.758 88.9 90)
 			(effects
@@
 			)
 		)
-		(property "Footprint" ""
+		(property "Footprint" "Resistor_SMD:R_0805_2012Metric_Pad1.20x1.40mm_HandSolder"
 			(at 114.935 196.723 90)
 			(effects
@@
 			)
 		)
-		(property "Footprint" ""
+		(property "Footprint" "Resistor_SMD:R_0805_2012Metric_Pad1.20x1.40mm_HandSolder"
 			(at 114.935 178.308 90)
 			(effects
@@
 			)
 		)
-		(property "Footprint" ""
+		(property "Footprint" "Resistor_SMD:R_0805_2012Metric_Pad1.20x1.40mm_HandSolder"
 			(at 90.17 144.018 90)
 			(effects
@@
 			)
 		)
-		(property "Footprint" ""
+		(property "Footprint" "Resistor_SMD:R_0805_2012Metric_Pad1.20x1.40mm_HandSolder"
 			(at 120.65 144.018 90)
 			(effects
@@
 			)
 		)
-		(property "Footprint" ""
+		(property "Footprint" "Resistor_SMD:R_0805_2012Metric_Pad1.20x1.40mm_HandSolder"
 			(at 90.17 105.918 90)
 			(effects
@@
 			)
 		)
-		(property "Footprint" ""
+		(property "Footprint" "Resistor_SMD:R_0805_2012Metric_Pad1.20x1.40mm_HandSolder"
 			(at 187.96 60.452 90)
 			(effects
@@
 			)
 		)
-		(property "Footprint" ""
+		(property "Footprint" "Resistor_SMD:R_0805_2012Metric_Pad1.20x1.40mm_HandSolder"
 			(at 153.162 137.16 90)
 			(effects
@@
 			)
 		)
-		(property "Footprint" ""
+		(property "Footprint" "Resistor_SMD:R_0805_2012Metric_Pad1.20x1.40mm_HandSolder"
 			(at 187.96 70.612 90)
 			(effects

Commit message: footprint setting in progress
Parts:
- C1, C3, C6, C7: value C -> 0,1uF; footprint (none) -> Capacitor_SMD:C_0805_2012Metric_Pad1.18x1.45mm_HandSolder
Changed lines of the file:
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@@
 			)
 		)
-		(property "Value" "C"
+		(property "Value" "0,1uF"
 			(at 62.23 222.2499 0)
 			(effects
@@
 			)
 		)
-		(property "Footprint" ""
+		(property "Footprint" "Capacitor_SMD:C_0805_2012Metric_Pad1.18x1.45mm_HandSolder"
 			(at 59.3852 224.79 0)
 			(effects
@@
 			)
 		)
-		(property "Value" "C"
+		(property "Value" "0,1uF"
 			(at 165.0999 154.94 0)
 			(effects
@@
 			)
 		)
-		(property "Footprint" ""
+		(property "Footprint" "Capacitor_SMD:C_0805_2012Metric_Pad1.18x1.45mm_HandSolder"
 			(at 167.64 157.7848 0)
 			(effects
@@
 			)
 		)
-		(property "Value" "C"
+		(property "Value" "0,1uF"
 			(at 157.48 247.6499 0)
 			(effects
@@
 			)
 		)
-		(property "Footprint" ""
+		(property "Footprint" "Capacitor_SMD:C_0805_2012Metric_Pad1.18x1.45mm_HandSolder"
 			(at 154.6352 250.19 0)
 			(effects
@@
 			)
 		)
-		(property "Value" "C"
+		(property "Value" "0,1uF"
 			(at 26.6701 134.62 0)
 			(effects
@@
 			)
 		)
-		(property "Footprint" ""
+		(property "Footprint" "Capacitor_SMD:C_0805_2012Metric_Pad1.18x1.45mm_HandSolder"
 			(at 24.13 131.7752 0)
 			(effects

Commit message: footprint setting in progress
Parts:
- D1: value LED -> white
- J3: footprint (none) -> Connector_PinHeader_2.54mm:PinHeader_1x04_P2.54mm_Vertical
- J4, J5: footprint (none) -> Connector_PinHeader_2.54mm:PinHeader_1x03_P2.54mm_Vertical
- J6: footprint (none) -> Connector_PinHeader_2.54mm:PinHeader_1x02_P2.54mm_Vertical
Changed lines of the file:
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@@
 			)
 		)
-		(property "Footprint" ""
+		(property "Footprint" "Connector_PinHeader_2.54mm:PinHeader_1x02_P2.54mm_Vertical"
 			(at 191.77 191.77 0)
 			(effects
@@
 			)
 		)
-		(property "Value" "LED"
+		(property "Value" "white"
 			(at 100.0124 244.475 0)
 			(effects
@@
 			)
 		)
-		(property "Footprint" ""
+		(property "Footprint" "Connector_PinHeader_2.54mm:PinHeader_1x03_P2.54mm_Vertical"
 			(at 191.77 182.245 0)
 			(effects
@@
 			)
 		)
-		(property "Footprint" ""
+		(property "Footprint" "Connector_PinHeader_2.54mm:PinHeader_1x03_P2.54mm_Vertical"
 			(at 191.77 167.64 0)
 			(effects
@@
 			)
 		)
-		(property "Footprint" ""
+		(property "Footprint" "Connector_PinHeader_2.54mm:PinHeader_1x04_P2.54mm_Vertical"
 			(at 191.77 151.13 0)
 			(effects

Commit message: footprint setting in progress
Parts:
- SW3, SW4, SW5, SW6: footprint (none) -> Button_Switch_THT:SW_PUSH_6mm_H9.5mm
- U1: value ~ -> CH32X035C8T6; footprint (none) -> Package_QFP:LQFP-48_7x7mm_P0.5mm
Changed lines of the file:
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@@
 			)
 		)
-		(property "Footprint" ""
+		(property "Footprint" "Button_Switch_THT:SW_PUSH_6mm_H9.5mm"
 			(at 163.83 170.18 0)
 			(effects
@@
 			)
 		)
-		(property "Footprint" ""
+		(property "Footprint" "Button_Switch_THT:SW_PUSH_6mm_H9.5mm"
 			(at 163.83 182.88 0)
 			(effects
@@
 			)
 		)
-		(property "Footprint" ""
+		(property "Footprint" "Button_Switch_THT:SW_PUSH_6mm_H9.5mm"
 			(at 163.83 176.53 0)
 			(effects
@@
 			)
 		)
-		(property "Footprint" ""
+		(property "Footprint" "Button_Switch_THT:SW_PUSH_6mm_H9.5mm"
 			(at 163.83 189.23 0)
 			(effects
@@
 			)
 		)
-		(property "Value" "~"
+		(property "Value" "CH32X035C8T6"
 			(at 66.04 145.4465 0)
 			(effects
@@
 					(size 1.27 1.27)
 				)
+				(hide yes)
 			)
 		)
-		(property "Footprint" ""
+		(property "Footprint" "Package_QFP:LQFP-48_7x7mm_P0.5mm"
 			(at 10.16 138.43 0)
 			(effects

Commit message: add quarz footprint
Parts:
- Y1: footprint (none) -> Crystal:Crystal_C38-LF_D3.0mm_L8.0mm_Horizontal

Commit message: add battery holder footprint
Parts:
- BT1: footprint (none) -> Battery:BatteryHolder_MYOUNG_BS-07-A1BJ001_CR2032
Changed lines of the file:
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@@
 			)
 		)
-		(property "Footprint" ""
+		(property "Footprint" "Battery:BatteryHolder_MYOUNG_BS-07-A1BJ001_CR2032"
 			(at 101.6 200.914 90)
 			(effects
