File: kicad/zxRebornClock/zxRebornClock.kicad_pcb (KiCad board)
At the start: 2 copper layers, 41.5 x 41.5 mm, 105 parts, among them J1 Jack DC, J2 USB_B_Micro, J3 Conn_01x04, J4 Conn_01x03, J5 Conn_01x03, J6 Conn_01x02, Q1 MMBTA42, Q10 MMBTA42, Q2 MMBTA42, Q3 MMBTA42, Q4 MMBTA42, Q5 MMBTA42, Q6 MMBTA42, Q7 MMBTA42, Q8 MMBTA42, Q9 MMBTA42, SW1 RESET, SW2 D, SW3 HH, SW4 MM, SW5 SS, SW6 F, U1 CH32X035C8T6, U10 TLP627, U2 AMS1117-3.3, U3 12V->200V, U4 USBLC6-4SC6, U5 DS1302, U6 ESP-12F, U7 TLP627, U8 TLP627, U9 TLP627, Y1 32768

Commit message: add edge
Parts:
- added H24: MountingHole, MountingHole:MountingHole_3.2mm_M3, F.Cu at (221.4, 106.7)
- added H25: MountingHole, MountingHole:MountingHole_3.2mm_M3, F.Cu at (221.4, 189.4)
- added H26: MountingHole, MountingHole:MountingHole_3.2mm_M3, F.Cu at (344.1, 189.4)
- added H27: MountingHole, MountingHole:MountingHole_3.2mm_M3, F.Cu at (344.1, 106.7)
Other:
- board size 41.5 x 41.5 mm -> 148.5 x 89.9 mm
- board text added: "for box G1024B"

Commit message: work in progress
Parts:
- moved VL1 209.1 mm to (252.1, 159.0), turned to 180 degrees
- moved VL2 208.7 mm to (272.6, 159.0), turned to 180 degrees
- moved VL3 208.2 mm to (293.0, 159.0), turned to 180 degrees
- moved VL4 208.0 mm to (313.9, 159.0), turned to 180 degrees
- moved J3 37.3 mm to (191.0, 62.8)
- moved J6 37.3 mm to (195.6, 62.8)
- moved U4 37.3 mm to (195.9, 70.0)
- moved J2 37.3 mm to (193.6, 56.3)

Commit message: fix footprint for 12v_200v
Parts:
- H1, H2, H3, H4, U3: moved to B.Cu
- moved U3 206.2 mm to (282.7, 150.1)
- moved H3 150.3 mm to (306.0, 119.0)
- moved H4 148.7 mm to (306.0, 113.0)
- moved H1 115.8 mm to (259.0, 137.9)
- moved H2 110.6 mm to (259.0, 132.3)
- moved VL1 10.0 mm to (252.1, 169.0)
- moved VL2 10.0 mm to (272.6, 169.0)
- moved VL3 10.0 mm to (293.0, 169.0)
- moved VL4 10.0 mm to (313.9, 169.0)

Commit message: work in progress
Parts:
- moved SW6 182.1 mm to (293.8, 176.2)
- moved SW5 177.0 mm to (284.2, 176.2)
- moved SW4 172.7 mm to (274.8, 176.2)
- moved SW3 169.2 mm to (265.2, 176.2)
- moved J1 62.5 mm to (222.5, 141.0)
- moved U2 57.6 mm to (73.2, 132.7)
- moved H3 37.1 mm to (343.0, 121.0)
- moved H4 37.1 mm to (343.0, 115.0)
- moved H1 37.1 mm to (296.0, 136.0)
- moved H2 37.1 mm to (296.0, 130.3)
- moved U3 37.0 mm to (319.7, 150.1)
Changed lines of the file:
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@@
 	(footprint "Connector_BarrelJack:BarrelJack_Horizontal"
 		(layer "F.Cu")
-		(at 169.361 108.115)
+		(at 222.5 141.0425)
 		(descr "DC Barrel Jack")
 		(tags "Power Jack")
@@
 	(footprint "Button_Switch_THT:SW_PUSH_6mm_H9.5mm"
 		(layer "F.Cu")
-		(at 125.681 89.13)
+		(at 274.75 176.25)
 		(descr "tactile push button, 6x6mm e.g. PHAP33xx series, height=9.5mm")
 		(tags "tact sw push 6mm")
@@
 	(footprint "Button_Switch_THT:SW_PUSH_6mm_H9.5mm"
 		(layer "F.Cu")
-		(at 125.681 106.23)
+		(at 293.75 176.25)
 		(descr "tactile push button, 6x6mm e.g. PHAP33xx series, height=9.5mm")
 		(tags "tact sw push 6mm")
@@
 	(footprint "Package_TO_SOT_SMD:SOT-223-3_TabPin2"
 		(layer "F.Cu")
-		(at 128.581 116.955)
+		(at 73.15 132.7)
 		(descr "module CMS SOT223 4 pins")
 		(tags "CMS SOT")
@@
 	(footprint "Button_Switch_THT:SW_PUSH_6mm_H9.5mm"
 		(layer "F.Cu")
-		(at 125.681 97.68)
+		(at 284.25 176.25)
 		(descr "tactile push button, 6x6mm e.g. PHAP33xx series, height=9.5mm")
 		(tags "tact sw push 6mm")
@@
 	(footprint "Button_Switch_THT:SW_PUSH_6mm_H9.5mm"
 		(layer "F.Cu")
-		(at 125.681 80.58)
+		(at 265.25 176.25)
 		(descr "tactile push button, 6x6mm e.g. PHAP33xx series, height=9.5mm")
 		(tags "tact sw push 6mm")
@@
 	(footprint "Library:12v_200v"
 		(layer "B.Cu")
-		(at 282.65165 150.149175)
+		(at 319.65165 150.149175)
 		(property "Reference" "U3"
 			(at 0 -22.699175 180)
@@
 	(footprint "TestPoint:TestPoint_THTPad_D4.0mm_Drill2.0mm"
 		(layer "B.Cu")
-		(at 259 132.3)
+		(at 296 130.35)
 		(descr "THT pad as test Point, diameter 4.0mm, hole diameter 2.0mm")
 		(tags "test point THT pad")
@@
 	(footprint "TestPoint:TestPoint_THTPad_D4.0mm_Drill2.0mm"
 		(layer "B.Cu")
-		(at 306 112.95)
+		(at 343 115)
 		(descr "THT pad as test Point, diameter 4.0mm, hole diameter 2.0mm")
 		(tags "test point THT pad")
@@
 	(footprint "TestPoint:TestPoint_THTPad_D4.0mm_Drill2.0mm"
 		(layer "B.Cu")
-		(at 259 137.95)
+		(at 296 136)
 		(descr "THT pad as test Point, diameter 4.0mm, hole diameter 2.0mm")
 		(tags "test point THT pad")
@@
 	(footprint "TestPoint:TestPoint_THTPad_D4.0mm_Drill2.0mm"
 		(layer "B.Cu")
-		(at 306 119)
+		(at 343 121.05)
 		(descr "THT pad as test Point, diameter 4.0mm, hole diameter 2.0mm")
 		(tags "test point THT pad")

Commit message: work in progress
Parts:
- BT1, C2, C4, J1, U1, U2, U5, U6, Y1: moved to B.Cu
- moved U6 217.8 mm to (344.5, 172.6), turned to 90 degrees
- moved BT1 162.0 mm to (233.5, 172.0), turned to 180 degrees
- moved Y1 159.2 mm to (241.6, 191.8)
- moved U1 158.0 mm to (271.2, 126.3), turned to 180 degrees
- moved U5 151.3 mm to (238.1, 191.6), turned to 90 degrees
- moved U2 149.7 mm to (222.8, 136.3), turned to 180 degrees
- moved R1 143.6 mm to (239.5, 138.5), turned to 90 degrees
- moved C4 89.9 mm to (232.5, 138.0), turned to 90 degrees
- moved D1 89.8 mm to (239.5, 134.5), turned to 90 degrees
- moved C5 85.8 mm to (235.0, 136.2), turned to 90 degrees
- moved C2 76.2 mm to (215.5, 138.5), turned to 180 degrees
- moved U10 37.1 mm to (99.5, 93.5)
- moved U7 37.1 mm to (99.5, 73.4)
- moved U8 37.1 mm to (99.5, 80.1)
- moved U9 37.1 mm to (99.5, 86.8)
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
Commit message: work in progress
Parts:
- moved D1 27.1 mm to (212.5, 132.0), turned to 180 degrees
- moved R1 23.9 mm to (216.5, 132.0), turned to 180 degrees
- moved C4 10.5 mm to (222.0, 138.3)
- moved C5 10.5 mm to (224.5, 136.5)
- moved U2 9.73 mm to (213.2, 137.0)
- moved C2 5.76 mm to (211.0, 142.0)
Changed lines of the file:
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@@
 	(footprint "Capacitor_SMD:C_0805_2012Metric_Pad1.18x1.45mm_HandSolder"
 		(layer "F.Cu")
-		(at 234.9825 136.1665 90)
+		(at 224.5 136.4625 90)
 		(descr "Capacitor SMD 0805 (2012 Metric), square (rectangular) end terminal, IPC_7351 nominal with elongated pad for handsoldering. (Body size source: IPC-SM-782 page 76, https://www.pcb-3d.com/wordpress/wp-content/uploads/ipc-sm-782a_amendment_1_and_2.pdf, https://docs.google.com/spreadsheets/d/1BsfQQcO9C6DZCsRaXUlFlo91Tg2WpOkGARC1WS5S8t0/edit?usp=sharing), generated with kicad-footprint-generator")
 		(tags "capacitor handsolder")
@@
 	(footprint "Resistor_SMD:R_0805_2012Metric_Pad1.20x1.40mm_HandSolder"
 		(layer "F.Cu")
-		(at 239.5 138.525 90)
+		(at 216.5 132 180)
 		(descr "Resistor SMD 0805 (2012 Metric), square (rectangular) end terminal, IPC_7351 nominal with elongated pad for handsoldering. (Body size source: IPC-SM-782 page 72, https://www.pcb-3d.com/wordpress/wp-content/uploads/ipc-sm-782a_amendment_1_and_2.pdf), generated with kicad-footprint-generator")
 		(tags "resistor handsolder")
 		(property "Reference" "R1"
-			(at 0 -1.65 90)
+			(at -3 0 360)
 			(layer "F.SilkS")
 			(effects
@@
 		)
 		(property "Value" "1,0K"
-			(at 0 1.65 90)
+			(at 0 1.65 360)
 			(layer "F.Fab")
 			(hide yes)
@@
 		)
 		(property "Footprint" "Resistor_SMD:R_0805_2012Metric_Pad1.20x1.40mm_HandSolder"
-			(at 0 0 90)
+			(at 0 0 180)
 			(unlocked yes)
 			(layer "F.Fab")
@@
 		)
 		(property "Datasheet" ""
-			(at 0 0 90)
+			(at 0 0 180)
 			(unlocked yes)
 			(layer "F.Fab")
@@
 		)
 		(property "Description" "Resistor"
-			(at 0 0 90)
+			(at 0 0 180)
 			(unlocked yes)
 			(layer "F.Fab")
@@
 		(attr smd)
 		(fp_line
-			(start -0.227064 -0.735)
-			(end 0.227064 -0.735)
+			(start -0.227064 0.735)
+			(end 0.227064 0.735)
 			(stroke
 				(width 0.12)
@@
 		)
 		(fp_line
-			(start -0.227064 0.735)
-			(end 0.227064 0.735)
+			(start -0.227064 -0.735)
+			(end 0.227064 -0.735)
 			(stroke
 				(width 0.12)
@@
 		)
 		(fp_line
-			(start 1.85 -0.95)
-			(end 1.85 0.95)
+			(start 1.85 0.95)
+			(end -1.85 0.95)
 			(stroke
 				(width 0.05)
@@
 		)
 		(fp_line
-			(start -1.85 -0.95)
-			(end 1.85 -0.95)
+			(start 1.85 -0.95)
+			(end 1.85 0.95)
 			(stroke
 				(width 0.05)
@@
 		)
 		(fp_line
-			(start 1.85 0.95)
-			(end -1.85 0.95)
+			(start -1.85 0.95)
+			(end -1.85 -0.95)
 			(stroke
 				(width 0.05)
@@
 		)
 		(fp_line
-			(start -1.85 0.95)
-			(end -1.85 -0.95)
+			(start -1.85 -0.95)
+			(end 1.85 -0.95)
 			(stroke
 				(width 0.05)
@@
 		)
 		(fp_line
-			(start 1 -0.625)
-			(end 1 0.625)
+			(start 1 0.625)
+			(end -1 0.625)
 			(stroke
 				(width 0.1)
@@
 		)
 		(fp_line
-			(start -1 -0.625)
-			(end 1 -0.625)
+			(start 1 -0.625)
+			(end 1 0.625)
 			(stroke
 				(width 0.1)
@@
 		)
 		(fp_line
-			(start 1 0.625)
-			(end -1 0.625)
+			(start -1 0.625)
+			(end -1 -0.625)
 			(stroke
 				(width 0.1)
@@
 		)
 		(fp_line
-			(start -1 0.625)
-			(end -1 -0.625)
+			(start -1 -0.625)
+			(end 1 -0.625)
 			(stroke
 				(width 0.1)
@@
 		)
 		(fp_text user "${REFERENCE}"
-			(at 0 0 90)
+			(at 0 0 360)
 			(layer "F.Fab")
 			(effects
@@
 		)
 		(pad "1" smd roundrect
-			(at -1 0 90)
+			(at -1 0 180)
 			(size 1.2 1.4)
 			(layers "F.Cu" "F.Paste" "F.Mask")
@@
 		)
 		(pad "2" smd roundrect
-			(at 1 0 90)
+			(at 1 0 180)
 			(size 1.2 1.4)
 			(layers "F.Cu" "F.Paste" "F.Mask")
@@
 	(footprint "LED_SMD:LED_0805_2012Metric_Pad1.15x1.40mm_HandSolder"
 		(layer "F.Cu")
-		(at 239.5 134.525 90)
+		(at 212.5 132 180)
 		(descr "LED SMD 0805 (2012 Metric), square (rectangular) end terminal, IPC_7351 nominal, (Body size source: https://docs.google.com/spreadsheets/d/1BsfQQcO9C6DZCsRaXUlFlo91Tg2WpOkGARC1WS5S8t0/edit?usp=sharing), generated with kicad-footprint-generator")
 		(tags "LED handsolder")
 		(property "Reference" "D1"
-			(at 0 -1.65 90)
+			(at 3 0 360)
 			(layer "F.SilkS")
 			(effects
@@
 		)
 		(property "Value" "white"
-			(at 0 1.65 90)
+			(at 0 1.65 360)
 			(layer "F.Fab")
 			(hide yes)
@@
 		)
 		(property "Footprint" "LED_SMD:LED_0805_2012Metric_Pad1.15x1.40mm_HandSolder"
-			(at 0 0 90)
+			(at 0 0 180)
 			(unlocked yes)
 			(layer "F.Fab")
@@
 		)
 		(property "Datasheet" ""
-			(at 0 0 90)
+			(at 0 0 180)
 			(unlocked yes)
 			(layer "F.Fab")
@@
 		)
 		(property "Description" "Light emitting diode"
-			(at 0 0 90)
+			(at 0 0 180)
 			(unlocked yes)
 			(layer "F.Fab")
@@
 		)
 		(fp_line
-			(start -1.86 -0.96)
-			(end -1.86 0.96)
+			(start -1.86 0.96)
+			(end 1 0.96)
 			(stroke
 				(width 0.12)
@@
 		)
 		(fp_line
-			(start -1.86 0.96)
-			(end 1 0.96)
+			(start -1.86 -0.96)
+			(end -1.86 0.96)
 			(stroke
 				(width 0.12)
@@
 		)
 		(fp_line
-			(start 1.85 -0.95)
-			(end 1.85 0.95)
+			(start 1.85 0.95)
+			(end -1.85 0.95)
 			(stroke
 				(width 0.05)
@@
 		)
 		(fp_line
-			(start -1.85 -0.95)
-			(end 1.85 -0.95)
+			(start 1.85 -0.95)
+			(end 1.85 0.95)
 			(stroke
 				(width 0.05)
@@
 		)
 		(fp_line
-			(start 1.85 0.95)
-			(end -1.85 0.95)
+			(start -1.85 0.95)
+			(end -1.85 -0.95)
 			(stroke
 				(width 0.05)
@@
 		)
 		(fp_line
-			(start -1.85 0.95)
-			(end -1.85 -0.95)
+			(start -1.85 -0.95)
+			(end 1.85 -0.95)
 			(stroke
 				(width 0.05)
@@
 		)
 		(fp_line
-			(start 1 -0.6)
-			(end -0.7 -0.6)
+			(start 1 0.6)
+			(end 1 -0.6)
 			(stroke
 				(width 0.1)
@@
 		)
 		(fp_line
-			(start -0.7 -0.6)
-			(end -1 -0.3)
+			(start 1 -0.6)
+			(end -0.7 -0.6)
 			(stroke
 				(width 0.1)
@@
 		)
 		(fp_line
-			(start -1 -0.3)
-			(end -1 0.6)
+			(start -0.7 -0.6)
+			(end -1 -0.3)
 			(stroke
 				(width 0.1)
@@
 		)
 		(fp_line
-			(start 1 0.6)
-			(end 1 -0.6)
+			(start -1 0.6)
+			(end 1 0.6)
 			(stroke
 				(width 0.1)
@@
 		)
 		(fp_line
-			(start -1 0.6)
-			(end 1 0.6)
+			(start -1 -0.3)
+			(end -1 0.6)
 			(stroke
 				(width 0.1)
@@
 		)
 		(fp_text user "${REFERENCE}"
-			(at 0 0 90)
+			(at 0 0 360)
 			(layer "F.Fab")
 			(effects
@@
 		)
 		(pad "1" smd roundrect
-			(at -1.025 0 90)
+			(at -1.025 0 180)
 			(size 1.15 1.4)
 			(layers "F.Cu" "F.Paste" "F.Mask")
@@
 		)
 		(pad "2" smd roundrect
-			(at 1.025 0 90)
+			(at 1.025 0 180)
 			(size 1.15 1.4)
 			(layers "F.Cu" "F.Paste" "F.Mask")
@@
 		(tags "Power Jack")
 		(property "Reference" "J1"
-			(at -8.45 -5.75 360)
+			(at -9.5 0 360)
 			(layer "B.SilkS")
 			(effects
@@
 		)
 		(property "Value" "Jack DC"
-			(at -6.2 5.5 360)
+			(at -6.2 5.5 0)
 			(layer "B.Fab")
+			(hide yes)
 			(effects
 				(font
@@
 		)
 		(fp_text user "${REFERENCE}"
-			(at -3 2.95 360)
+			(at -3 2.95 0)
 			(layer "B.Fab")
+			(hide yes)
 			(effects
 				(font
@@
 	(footprint "Package_TO_SOT_SMD:SOT-223-3_TabPin2"
 		(layer "B.Cu")
-		(at 222.85 136.3 180)
+		(at 213.15 137 180)
 		(descr "module CMS SOT223 4 pins")
 		(tags "CMS SOT")
 		(property "Reference" "U2"
-			(at 0 4.5 360)
+			(at 0 0 90)
 			(layer "B.SilkS")
 			(effects
@@
 			(at 0 0 90)
 			(layer "B.Fab")
+			(hide yes)
 			(effects
 				(font
@@
 	(footprint "Capacitor_SMD:C_0805_2012Metric_Pad1.18x1.45mm_HandSolder"
 		(layer "B.Cu")
-		(at 215.5375 138.5 180)
+		(at 210.9625 142 180)
 		(descr "Capacitor SMD 0805 (2012 Metric), square (rectangular) end terminal, IPC_7351 nominal with elongated pad for handsoldering. (Body size source: IPC-SM-782 page 76, https://www.pcb-3d.com/wordpress/wp-content/uploads/ipc-sm-782a_amendment_1_and_2.pdf, https://docs.google.com/spreadsheets/d/1BsfQQcO9C6DZCsRaXUlFlo91Tg2WpOkGARC1WS5S8t0/edit?usp=sharing), generated with kicad-footprint-generator")
 		(tags "capacitor handsolder")
 		(property "Reference" "C2"
-			(at 0 1.68 360)
+			(at -3.5375 0 360)
 			(layer "B.SilkS")
 			(effects
@@
 	(footprint "Capacitor_THT:CP_Radial_D8.0mm_P3.50mm"
 		(layer "B.Cu")
-		(at 232.5 138 90)
+		(at 222.0175 138.296 90)
 		(descr "CP, Radial series, Radial, pin pitch=3.50mm, , diameter=8mm, Electrolytic Capacitor")
 		(tags "CP Radial series Radial pin pitch 3.50mm  diameter 8mm Electrolytic Capacitor")

Commit message: work in progress
Parts:
- J2: moved to B.Cu
- moved R31 207.6 mm to (274.6, 208.8)
- moved R32 206.9 mm to (274.6, 210.8)
- moved R33 206.1 mm to (274.6, 212.8)
- moved R30 190.2 mm to (274.6, 206.8)
- moved J2 91.9 mm to (271.0, 105.8)

Commit message: work in progress
Parts:
- R30, R31, R32, R33: moved to B.Cu
- moved R33 36.9 mm to (297.0, 183.5), turned to 180 degrees
- moved R32 30.2 mm to (287.5, 183.5), turned to 180 degrees
- moved R31 25.5 mm to (278.0, 183.5), turned to 180 degrees
- moved R30 24.1 mm to (268.5, 183.5), turned to 180 degrees
