File: kicad/zxRebornClock/zxRebornClock.kicad_pcb (KiCad board)
At the start: 2 copper layers, 148.5 x 89.9 mm, 109 parts, among them J1 Jack DC, J2 USB_B_Micro, J3 Conn_01x04, J4 Conn_01x03, J5 Conn_01x03, J6 Conn_01x02, Q1 MMBTA42, Q10 MMBTA42, Q2 MMBTA42, Q3 MMBTA42, Q4 MMBTA42, Q5 MMBTA42, Q6 MMBTA42, Q7 MMBTA42, Q8 MMBTA42, Q9 MMBTA42, SW1 RESET, SW2 D, SW3 HH, SW4 MM, SW5 SS, SW6 F, U1 CH32X035C8T6, U10 TLP627, U2 AMS1117-3.3, U3 12V->200V, U4 USBLC6-4SC6, U5 DS1302, U6 ESP-12F, U7 TLP627, U8 TLP627, U9 TLP627, Y1 32768

Commit message: work in progress
Parts:
- R35, R36, R37, R38, R39, R40, R41, R42, R43, R44: moved to B.Cu
- moved R41 167.6 mm to (252.0, 179.5), turned to 180 degrees
- moved R42 166.8 mm to (252.0, 181.5), turned to 180 degrees
- moved R43 166.1 mm to (252.0, 183.5), turned to 180 degrees
- moved R44 165.4 mm to (252.0, 185.5), turned to 180 degrees
- moved R40 157.1 mm to (252.0, 187.5), turned to 180 degrees
- moved R35 154.8 mm to (252.0, 169.5), turned to 180 degrees
- moved R36 154.2 mm to (252.0, 171.5), turned to 180 degrees
- moved R37 153.5 mm to (252.0, 173.5), turned to 180 degrees
- moved R38 152.9 mm to (252.0, 175.5), turned to 180 degrees
- moved R39 152.2 mm to (252.0, 177.5), turned to 180 degrees

Commit message: work in progress
Parts:
- moved R11 132.1 mm to (151.5, 181.0), turned to 180 degrees
- moved R25 122.3 mm to (165.0, 181.0), turned to 180 degrees
- moved R24 116.9 mm to (165.0, 172.5), turned to 180 degrees
- moved R6 116.5 mm to (151.5, 179.0)
- moved R23 112.0 mm to (165.0, 164.5), turned to 180 degrees
- moved R5 111.1 mm to (151.5, 170.5)
- moved R22 107.6 mm to (165.0, 157.0), turned to 180 degrees
- moved R20 107.5 mm to (165.0, 179.0)
- moved R4 106.2 mm to (151.5, 162.5)
- moved R21 103.3 mm to (165.0, 149.5), turned to 180 degrees
- moved R19 102.3 mm to (165.0, 170.5)
- moved R3 101.8 mm to (151.5, 155.0)
- moved R10 98.8 mm to (151.5, 172.5), turned to 180 degrees
- moved R18 97.5 mm to (165.0, 162.5)
- moved R2 97.4 mm to (151.5, 147.5)
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
Commit message: work in progress
Parts:
- Q1, Q10, Q2, Q3, Q4, Q5, Q6, Q7, Q8, Q9, R10, R11, R16, R17, R18, R19, R2, R20, R21, R22, R23, R24, R25, R28, R3, R4, R45, R46, R47, R48, R5, R6, R7, R8, R9, RV1, U10, U7, U8, U9: moved to B.Cu
- moved U7 151.7 mm to (243.5, 121.0), turned to 180 degrees
- moved U8 151.5 mm to (243.5, 127.0), turned to 180 degrees
- moved U9 151.3 mm to (243.5, 133.0), turned to 180 degrees
- moved U10 151.1 mm to (243.5, 139.0), turned to 180 degrees
- moved R10 141.6 mm to (287.5, 133.0), turned to 0 degrees
- moved R11 141.6 mm to (287.5, 141.5), turned to 0 degrees
- moved R2 141.6 mm to (287.5, 108.0), turned to 180 degrees
- moved R3 141.6 mm to (287.5, 115.5), turned to 180 degrees
- moved R4 141.6 mm to (287.5, 123.0), turned to 180 degrees
- moved R5 141.6 mm to (287.5, 131.0), turned to 180 degrees
- moved R6 141.6 mm to (287.5, 139.5), turned to 180 degrees
- moved R7 141.6 mm to (287.5, 110.0), turned to 0 degrees
- moved R8 141.6 mm to (287.5, 117.5), turned to 0 degrees
- moved R9 141.6 mm to (287.5, 125.0), turned to 0 degrees
- moved Q1 133.8 mm to (283.4, 109.0), turned to 180 degrees
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
Commit message: work in progress
Parts:
- moved J6 81.6 mm to (151.5, 131.5)
- moved J3 81.2 mm to (147.5, 131.4)
- moved U4 45.7 mm to (241.4, 74.5)
- moved J5 19.8 mm to (143.5, 131.4)
- moved J4 19.5 mm to (139.5, 131.4)
Changed lines of the file:
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@@
 	(footprint "Connector_PinHeader_2.54mm:PinHeader_1x03_P2.54mm_Vertical"
 		(layer "F.Cu")
-		(at 152.031 113.55)
+		(at 143.5 131.42)
 		(descr "Through hole straight pin header, 1x03, 2.54mm pitch, single row")
 		(tags "Through hole pin header THT 1x03 2.54mm single row")
@@
 			(at 0 7.41 0)
 			(layer "F.Fab")
+			(hide yes)
 			(effects
 				(font
@@
 			(at 0 2.54 90)
 			(layer "F.Fab")
+			(hide yes)
 			(effects
 				(font
@@
 	(footprint "Connector_PinHeader_2.54mm:PinHeader_1x04_P2.54mm_Vertical"
 		(layer "F.Cu")
-		(at 190.9625 62.775)
+		(at 147.5 131.38)
 		(descr "Through hole straight pin header, 1x04, 2.54mm pitch, single row")
 		(tags "Through hole pin header THT 1x04 2.54mm single row")
@@
 			(at 0 9.95 0)
 			(layer "F.Fab")
+			(hide yes)
 			(effects
 				(font
@@
 			(at 0 3.81 90)
 			(layer "F.Fab")
+			(hide yes)
 			(effects
 				(font
@@
 	(footprint "Package_TO_SOT_SMD:SOT-23-6"
 		(layer "F.Cu")
-		(at 195.8625 70.05)
+		(at 241.3625 74.55)
 		(descr "SOT, 6 Pin (JEDEC MO-178 Var AB https://www.jedec.org/document_search?search_api_views_fulltext=MO-178), generated with kicad-footprint-generator ipc_gullwing_generator.py")
 		(tags "SOT TO_SOT_SMD")
@@
 	(footprint "Connector_PinHeader_2.54mm:PinHeader_1x02_P2.54mm_Vertical"
 		(layer "F.Cu")
-		(at 195.6125 62.775)
+		(at 151.5 131.46)
 		(descr "Through hole straight pin header, 1x02, 2.54mm pitch, single row")
 		(tags "Through hole pin header THT 1x02 2.54mm single row")
@@
 			(at 0 4.87 0)
 			(layer "F.Fab")
+			(hide yes)
 			(effects
 				(font
@@
 			(at 0 1.27 90)
 			(layer "F.Fab")
+			(hide yes)
 			(effects
 				(font
@@
 	(footprint "Connector_PinHeader_2.54mm:PinHeader_1x03_P2.54mm_Vertical"
 		(layer "F.Cu")
-		(at 147.381 113.55)
+		(at 139.5 131.42)
 		(descr "Through hole straight pin header, 1x03, 2.54mm pitch, single row")
 		(tags "Through hole pin header THT 1x03 2.54mm single row")
@@
 			(at 0 7.41 0)
 			(layer "F.Fab")
+			(hide yes)
 			(effects
 				(font
@@
 			(at 0 2.54 90)
 			(layer "F.Fab")
+			(hide yes)
 			(effects
 				(font

Commit message: work in progress
Parts:
- R26, R27, R34, R49, R50: moved to B.Cu
- moved R26 240.1 mm to (347.0, 179.0), turned to 180 degrees
- moved R27 235.2 mm to (343.0, 179.0), turned to 180 degrees
- moved R34 217.2 mm to (335.0, 155.5)
- moved R49 214.0 mm to (343.0, 155.5), turned to 180 degrees
- moved R50 209.2 mm to (339.0, 155.5), turned to 180 degrees
- moved U6 5.50 mm to (344.5, 167.1)

Commit message: work in progress
Parts:
- moved R12 231.5 mm to (347.5, 135.0)
- moved R13 231.2 mm to (347.5, 137.0)
- moved R14 230.9 mm to (347.5, 139.0)
- moved R15 230.6 mm to (347.5, 141.0)
- moved D2 190.6 mm to (351.5, 135.0), turned to 180 degrees
- moved D3 190.3 mm to (351.5, 137.0), turned to 180 degrees
- moved D4 190.0 mm to (351.5, 139.0), turned to 180 degrees
- moved D5 189.7 mm to (351.5, 141.0), turned to 180 degrees
- moved C6 182.1 mm to (329.5, 166.5), turned to -90 degrees

Commit message: work in progress
Parts:
- C1, J5, J6: moved to B.Cu
- moved J5 210.4 mm to (352.6, 155.0), turned to 90 degrees
- moved J6 192.3 mm to (337.5, 180.0), turned to 90 degrees
- moved C1 100.7 mm to (256.5, 118.0)
- moved VL4 0.35 mm to (313.5, 169.0)

Commit message: work in progress
Parts:
- J3, J4: moved to B.Cu
- moved R29 93.4 mm to (219.5, 115.0)
- moved J4 92.3 mm to (227.9, 105.0), turned to -90 degrees
- moved SW1 87.7 mm to (226.6, 119.5)
- moved SW2 87.0 mm to (226.6, 115.0)
- moved J3 64.9 mm to (211.0, 117.9), turned to 180 degrees
- moved C7 61.3 mm to (219.5, 119.5), turned to 180 degrees
