File: kicad/zxRebornClock/zxRebornClock.kicad_pcb (KiCad board)
At the start: 2 copper layers, 148.5 x 90 mm, 111 parts, among them J1 Jack DC, J2 USB_B_Micro, J3 Conn_01x04, J4 Conn_01x03, J5 Conn_01x03, J6 Conn_01x02, Q1 MMBTA42, Q10 MMBTA42, Q2 MMBTA42, Q3 MMBTA42, Q4 MMBTA42, Q5 MMBTA42, Q6 MMBTA42, Q7 MMBTA42, Q8 MMBTA42, Q9 MMBTA42, SW1 RESET, SW2 D, SW3 HH, SW4 MM, SW5 SS, SW6 F, U1 CH32X035C8T6, U10 TLP627, U2 AMS1117-3.3, U3 12V->200V, U4 USBLC6-4SC6, U5 DS1302, U6 ESP-12F, U7 TLP627, U8 TLP627, U9 TLP627, Y1 32768

Commit message: work in progress
Parts:
- moved C5 4.75 mm to (41.5, 113.5)
Routing:
- net /VCC: track 128.4 -> 146.6 mm, vias 4 -> 5
- net GND: track 356.2 -> 370.0 mm, vias 12 -> 16
- net /12V: track 29.7 -> 18.4 mm
- net Net-(D1-A): track 0.00 -> 7.41 mm
Changed lines of the file:
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@@
 	(footprint "Capacitor_SMD:C_0805_2012Metric_Pad1.18x1.45mm_HandSolder"
 		(layer "F.Cu")
-		(at 46.25 113.4125 90)
+		(at 41.5 113.4625 90)
 		(descr "Capacitor SMD 0805 (2012 Metric), square (rectangular) end terminal, IPC_7351 nominal with elongated pad for handsoldering. (Body size source: IPC-SM-782 page 76, https://www.pcb-3d.com/wordpress/wp-content/uploads/ipc-sm-782a_amendment_1_and_2.pdf, https://docs.google.com/spreadsheets/d/1BsfQQcO9C6DZCsRaXUlFlo91Tg2WpOkGARC1WS5S8t0/edit?usp=sharing), generated with kicad-footprint-generator")
 		(tags "capacitor handsolder")
@@
 	(segment
 		(start 43.7675 111.746)
-		(end 75.496 111.746)
+		(end 55.25 111.746)
 		(width 0.5)
 		(layer "F.Cu")
@@
 	)
 	(segment
-		(start 164.75 91.95)
-		(end 177.75 104.95)
+		(start 35 109.225)
+		(end 35.275 108.95)
 		(width 0.5)
 		(layer "F.Cu")
@@
 	)
 	(segment
-		(start 38.25 124.95)
-		(end 42.8 129.5)
+		(start 55.25 129.5)
+		(end 63.5 129.5)
+		(width 0.5)
+		(layer "F.Cu")
+		(net 1)
+	)
+	(segment
+		(start 164.75 91.95)
+		(end 177.75 104.95)
 		(width 0.5)
 		(layer "F.Cu")
@@
 	)
 	(segment
+		(start 35 111.75)
+		(end 35 109.225)
+		(width 0.5)
+		(layer "F.Cu")
+		(net 1)
+	)
+	(segment
 		(start 136 129.5)
 		(end 144 129.5)
@@
 	)
 	(segment
+		(start 55.25 111.746)
+		(end 75.496 111.746)
+		(width 0.5)
+		(layer "F.Cu")
+		(net 1)
+	)
+	(segment
 		(start 92.71 126.21)
 		(end 92.71 122.79)
@@
 	)
 	(segment
-		(start 44.3965 112.375)
+		(start 43.0885 112.425)
 		(end 43.7675 111.746)
 		(width 0.5)
@@
 	)
 	(segment
-		(start 46.25 112.375)
-		(end 44.3965 112.375)
+		(start 111.1 120.1)
+		(end 107.4 120.1)
 		(width 0.5)
 		(layer "F.Cu")
@@
 	)
 	(segment
-		(start 111.1 120.1)
-		(end 107.4 120.1)
+		(start 41.5 112.425)
+		(end 43.0885 112.425)
 		(width 0.5)
 		(layer "F.Cu")
@@
 	)
 	(segment
-		(start 42.8 129.5)
-		(end 63.5 129.5)
+		(start 113.4 120.1)
+		(end 112.25 121.25)
 		(width 0.5)
 		(layer "F.Cu")
@@
 	)
 	(segment
-		(start 113.4 120.1)
-		(end 112.25 121.25)
+		(start 35 116.5)
+		(end 35 111.75)
 		(width 0.5)
 		(layer "F.Cu")
@@
 	)
 	(via
+		(at 35 116.5)
+		(size 1)
+		(drill 0.4)
+		(layers "F.Cu" "B.Cu")
+		(net 1)
+	)
+	(via
+		(at 55.25 111.746)
+		(size 1)
+		(drill 0.4)
+		(layers "F.Cu" "B.Cu")
+		(net 1)
+	)
+	(via
 		(at 128 129.5)
 		(size 1)
@@
 	)
 	(via
+		(at 55.25 129.5)
+		(size 1)
+		(drill 0.4)
+		(layers "F.Cu" "B.Cu")
+		(net 1)
+	)
+	(via
 		(at 157.5 140.5)
 		(size 1)
@@
 	)
 	(via
+		(at 35 111.75)
+		(size 1)
+		(drill 0.4)
+		(layers "F.Cu" "B.Cu")
+		(net 1)
+	)
+	(via
 		(at 63.5 129.5)
 		(size 1)
@@
 	)
 	(segment
-		(start 75.575 105.825)
-		(end 74 104.25)
-		(width 0.2)
+		(start 35.1 111.65)
+		(end 35 111.75)
+		(width 0.5)
 		(layer "B.Cu")
 		(net 1)
 	)
 	(segment
-		(start 93.5 130)
-		(end 93.5 129.925)
+		(start 38.05 111.65)
+		(end 35.1 111.65)
 		(width 0.5)
 		(layer "B.Cu")
@@
 	)
 	(segment
-		(start 35.3625 122.6375)
-		(end 37.675 124.95)
+		(start 75.575 105.825)
+		(end 74 104.25)
+		(width 0.2)
+		(layer "B.Cu")
+		(net 1)
+	)
+	(segment
+		(start 93.5 130)
+		(end 93.5 129.925)
 		(width 0.5)
 		(layer "B.Cu")
@@
 	)
 	(segment
-		(start 37.675 124.95)
-		(end 38.25 124.95)
+		(start 87.55 129.05)
+		(end 88 129.5)
 		(width 0.5)
 		(layer "B.Cu")
@@
 	)
 	(segment
-		(start 87.55 129.05)
-		(end 88 129.5)
+		(start 157.5 140.5)
+		(end 155.75 138.75)
 		(width 0.5)
 		(layer "B.Cu")
@@
 	)
 	(segment
-		(start 157.5 140.5)
-		(end 155.75 138.75)
+		(start 38.25 124.95)
+		(end 37.675 124.95)
 		(width 0.5)
 		(layer "B.Cu")
@@
 	)
 	(segment
-		(start 31.675 118.95)
-		(end 35.3625 122.6375)
+		(start 37.675 124.95)
+		(end 31.675 118.95)
 		(width 0.5)
 		(layer "B.Cu")
@@
 	)
 	(segment
+		(start 55.25 111.746)
+		(end 55.25 129.5)
+		(width 0.5)
+		(layer "B.Cu")
+		(net 1)
+	)
+	(segment
 		(start 127.6 127.875)
 		(end 127.6 129.1)
@@
 	)
 	(segment
+		(start 34.125 116.5)
+		(end 35 116.5)
+		(width 0.5)
+		(layer "B.Cu")
+		(net 1)
+	)
+	(segment
 		(start 135.55 129.05)
 		(end 136 129.5)
@@
 	)
 	(segment
+		(start 31.675 118.95)
+		(end 34.125 116.5)
+		(width 0.5)
+		(layer "B.Cu")
+		(net 1)
+	)
+	(segment
 		(start 155.75 134.25)
 		(end 155.75 132.45)
@@
 	)
 	(segment
-		(start 46.25 114.45)
-		(end 44.5635 114.45)
+		(start 168.25 111.95)
+		(end 168.25 113.95)
 		(width 0.5)
 		(layer "F.Cu")
@@
 	)
 	(segment
-		(start 168.25 111.95)
-		(end 168.25 113.95)
+		(start 31.75 106)
+		(end 39.25 106)
 		(width 0.5)
 		(layer "F.Cu")
@@
 	)
 	(segment
+		(start 39.25 106)
+		(end 39.25 108.95)
+		(width 0.5)
+		(layer "F.Cu")
+		(net 3)
+	)
+	(segment
 		(start 157.5 144.5)
 		(end 157.5 148.5)
@@
 	)
 	(segment
-		(start 44.5635 114.45)
+		(start 43.0215 114.5)
 		(end 43.7675 115.246)
 		(width 0.5)
@@
 	)
 	(segment
+		(start 41.5 114.5)
+		(end 43.0215 114.5)
+		(width 0.5)
+		(layer "F.Cu")
+		(net 3)
+	)
+	(segment
 		(start 168.25 115.95)
 		(end 168.25 117.95)
@@
 	)
 	(via
+		(at 31.75 106)
+		(size 1)
+		(drill 0.4)
+		(layers "F.Cu" "B.Cu")
+		(net 3)
+	)
+	(via
 		(at 165.75 121.75)
 		(size 1)
@@
 	)
 	(segment
+		(start 31.75 113.95)
+		(end 31.75 106)
+		(width 0.5)
+		(layer "B.Cu")
+		(net 3)
+	)
+	(segment
 		(start 165.75 132.45)
 		(end 164.75 133.45)
@@
 	)
 	(segment
-		(start 45.5 119.5)
-		(end 48 119.5)
+		(start 42 124.95)
+		(end 36 118.95)
 		(width 0.5)
 		(layer "B.Cu")
@@
 	)
 	(segment
-		(start 35.35 118.95)
-		(end 38.05 116.25)
+		(start 36 118.95)
+		(end 33.75 118.95)
 		(width 0.5)
 		(layer "B.Cu")
@@
 	)
 	(segment
-		(start 36 118.95)
-		(end 33.75 118.95)
+		(start 44.25 124.95)
+		(end 42 124.95)
 		(width 0.5)
 		(layer "B.Cu")
@@
 	)
 	(segment
-		(start 38.05 116.25)
-		(end 42.25 116.25)
+		(start 35.35 118.95)
+		(end 38.05 116.25)
 		(width 0.5)
 		(layer "B.Cu")
@@
 	)
 	(segment
-		(start 42 124.95)
-		(end 36 118.95)
+		(start 37.25 107.25)
+		(end 37.25 108.95)
 		(width 0.5)
-		(layer "B.Cu")
-		(net 4)
+		(layer "F.Cu")
+		(net 6)
 	)
 	(segment
-		(start 42.25 116.25)
-		(end 45.5 119.5)
+		(start 33.225 108.95)
+		(end 33.225 107.275)
 		(width 0.5)
-		(layer "B.Cu")
-		(net 4)
+		(layer "F.Cu")
+		(net 6)
 	)
 	(segment
-		(start 44.25 124.95)
-		(end 42 124.95)
+		(start 33.225 107.275)
+		(end 33.25 107.25)
 		(width 0.5)
-		(layer "B.Cu")
-		(net 4)
+		(layer "F.Cu")
+		(net 6)
+	)
+	(segment
+		(start 33.25 107.25)
+		(end 37.25 107.25)
+		(width 0.5)
+		(layer "F.Cu")
+		(net 6)
 	)
 	(segment

Commit message: work in progress
Parts:
- moved H2 49.1 mm to (165.0, 97.3), turned to 180 degrees
- moved H3 49.0 mm to (117.5, 111.0)
- moved H4 49.0 mm to (117.5, 105.0)
- moved H1 47.5 mm to (165.0, 91.7), turned to 180 degrees
Routing:
- net /12V: track 18.4 -> 152.9 mm, vias 0 -> 2
- net /200V: track 0.00 -> 37.7 mm
- net GND: track 370.0 -> 404.3 mm
- net /K9: track 67.5 -> 73.5 mm
- net /K0: track 75.8 -> 81.5 mm
- net /K6: track 83.9 -> 89.5 mm
- net /K8: track 63.2 -> 65.6 mm

Commit message: work in progress
Connections:
- U1 pad 19: unconnected-(U1-PC7-Pad19) -> /DS_CLK
- U1 pad 20: /DS_CLK -> /DS_IO
- U1 pad 21: /B_HH -> /DS_CE
Routing:
- net /DS_CE: track 0.00 -> 68.9 mm
- net /DS_CLK: track 0.00 -> 68.1 mm
- net /DS_IO: track 0.00 -> 68.0 mm

Commit message: work in progress
Parts:
- moved D2 128.5 mm to (65.5, 42.0)
- moved D3 128.5 mm to (65.5, 44.0)
- moved D4 128.5 mm to (65.5, 46.0)
- moved D5 128.5 mm to (65.5, 48.0)
- moved R12 128.5 mm to (61.5, 42.0)
- moved R13 128.5 mm to (61.5, 44.0)
- moved R14 128.5 mm to (61.5, 46.0)
- moved R15 128.5 mm to (61.5, 48.0)
- moved Y1 5.20 mm to (63.5, 163.5), turned to -90 degrees
- moved H2 0.35 mm to (165.0, 97.0)
- moved H1 0.20 mm to (165.0, 91.5)
Connections:
- U1 pad 22: /B_MM -> /ESP_EN
Routing:
- net /VCC: track 146.6 -> 298.0 mm
- net GND: track 404.3 -> 486.0 mm
- net Net-(BT1-+): track 0.00 -> 31.6 mm
- net Net-(U5-X2): track 0.00 -> 10.8 mm
- net Net-(U5-X1): track 0.00 -> 7.48 mm

Commit message: work in progress
Routing:
- net /ESP_EN: track 4.87 -> 185.9 mm, vias 0 -> 1
- net /ESP_TX: track 6.44 -> 185.7 mm, vias 0 -> 2
- net /ESP_RX: track 5.12 -> 180.6 mm, vias 0 -> 2
- net /12V: track 152.9 -> 155.1 mm

Commit message: work in progress
Parts:
- moved C3 56.3 mm to (35.5, 60.5)
- moved J2 56.3 mm to (28.0, 55.2)
- moved U4 56.3 mm to (31.1, 60.6)
- moved SW3 40.5 mm to (87.0, 92.0)
- moved SW4 40.5 mm to (96.5, 92.0)
- moved SW5 40.5 mm to (106.0, 92.0)
- moved SW6 40.5 mm to (115.5, 92.0)
- moved C7 39.4 mm to (13.5, 68.5)
- moved R29 39.4 mm to (13.5, 64.0)
- moved SW1 39.4 mm to (20.6, 68.5)
- moved SW2 39.4 mm to (20.6, 64.0)
- moved J3 37.7 mm to (2.50, 72.4)
- moved J4 35.8 mm to (39.9, 47.5)
- moved R30 35.0 mm to (90.2, 93.8), turned to -90 degrees
- moved R31 35.0 mm to (99.8, 93.8), turned to -90 degrees
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Connections:
- U1 pad 23: /B_SS -> unconnected-(U1-PB3-Pad23)
- U1 pad 24: /B_F -> unconnected-(U1-PB4-Pad24)
- U1 pad 38: unconnected-(U1-PC14-Pad38) -> /B_HH
- U1 pad 39: unconnected-(U1-PC15-Pad39) -> /B_MM
- U1 pad 40: unconnected-(U1-PA8-Pad40) -> /B_SS
- U1 pad 41: unconnected-(U1-PA9-Pad41) -> /B_F
Routing:
- net /VCC: track 298.0 -> 379.0 mm, vias 5 -> 7
- net /B_F: track 0.00 -> 51.6 mm
- net /B_SS: track 0.00 -> 41.8 mm
- net /B_MM: track 0.00 -> 32.1 mm
- net /B_HH: track 0.00 -> 22.4 mm
- net Net-(R33-Pad2): track 0.00 -> 8.78 mm
- net Net-(R32-Pad2): track 0.00 -> 8.78 mm
- net Net-(R31-Pad2): track 0.00 -> 8.78 mm
- net Net-(R30-Pad2): track 0.00 -> 8.78 mm
Other:
- board size 148.5 x 90 mm -> 155.2 x 118.5 mm

Commit message: work in progress
Parts:
- C3: moved to F.Cu
- moved D2 88.6 mm to (-3.73, 97.2)
- moved D3 88.6 mm to (-3.77, 99.2)
- moved D4 88.6 mm to (-3.77, 101.2)
- moved D5 88.6 mm to (-3.77, 103.2)
- moved R12 88.6 mm to (-7.75, 97.2)
- moved R13 88.6 mm to (-7.75, 99.2)
- moved R14 88.6 mm to (-7.75, 101.2)
- moved R15 88.6 mm to (-7.75, 103.2)
- moved J4 56.3 mm to (4.42, 91.2)
- moved J2 50.1 mm to (69.1, 83.8)
- moved U4 49.2 mm to (69.5, 91.1), turned to -90 degrees
- moved C3 45.9 mm to (69.8, 91.0), turned to -90 degrees
Connections:
- U4 pad 1: /DOWNLOAD -> /UDM
- U4 pad 3: /UDM -> /DOWNLOAD
- U4 pad 4: /UDM -> /DOWNLOAD
- U4 pad 6: /DOWNLOAD -> /UDM
Routing:
- net GND: track 486.0 -> 534.0 mm, vias 16 -> 18
- net /12V: track 155.1 -> 202.6 mm
- net /VCC: track 379.0 -> 397.2 mm, vias 7 -> 8
- net /DOWNLOAD: track 0.00 -> 13.5 mm
- net /UDM: track 0.00 -> 12.8 mm
Other:
- board size 155.2 x 118.5 mm -> 148.5 x 90 mm

Commit message: work in progress
Parts:
- moved R29 76.3 mm to (87.5, 82.5), turned to 180 degrees
- moved C7 74.7 mm to (72.7, 114.0), turned to 45 degrees
- moved SW1 72.8 mm to (77.2, 114.3), turned to 45 degrees
- moved SW2 62.6 mm to (80.4, 82.5), turned to 180 degrees
Routing:
- net /RST: track 0.00 -> 13.7 mm
- net /VCC: track 397.2 -> 407.3 mm
- net /12V: track 202.6 -> 206.6 mm
- net GND: track 534.0 -> 536.0 mm
